File: boxes/electrons/NB3_body/NB3_body.kicad_sch (KiCad schematic)
At the start: 44 parts, among them J1 Conn_02x05_Counter_Clockwise, J10 JST SH 4-way Socket, J12 Conn_02x03_Top_Bottom, J13 Conn_02x03_Top_Bottom, J14 Conn_02x05_Counter_Clockwise, J15 Conn_02x05_Counter_Clockwise, J2 Conn_02x05_Counter_Clockwise, J3 Conn_02x05_Counter_Clockwise, J4 Conn_02x05_Counter_Clockwise, J5 Conn_02x05_Counter_Clockwise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

Commit message: Work on PCBs (v1 and v2)
Parts:
- added H31, H32: MountingHole, MountingHole:MountingHole_2.7mm_M2.5_ISO7380_Pad, symbol Mechanical:MountingHole
- added J11: JST SH 4-way Socket, NB3_body:Connector_S4B-PH-SM4-TB(LF)(SN), symbol NB3_body:Connector_S4B-PH-SM4-TB(LF)(SN)
Connections:
- net +5V: now also J11.1, J11.2
- net GND: now also J11.3, J11.4
Other:
- moved on the sheet: H1, H10, H11, H12, H13, H14, H15, H16, H17, H18, H19, H2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

Commit message: Update NB3 Body (rev 6)
Parts:
- J12, J13: footprint Connector_PinHeader_2.54mm:PinHeader_2x03_P2.54mm_Vertical_SMD -> Connector_PinHeader_2.54mm:PinHeader_2x03_P2.54mm_Vertical
Other:
- moved on the sheet: J1, J10, J11, J14, J15, J3, J5, J7, J8
